File: kicad/plytka_0_1.kicad_pcb (KiCad board)
At the start: 2 copper layers, 57 parts, among them P1 LED_SUPPY, P10 LV_POWER, P2 230V, P3 MEAN_WELL, P4 DS18b20_1, P5 DS18b20_2, P6 LEDs, P7 ADC(NC), P8 ESP_PIN1(NC), P9 ESP_PINS2(NC)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

Commit message: almost final PCB
Parts:
- removed P10: LV_POWER, Pin_Headers:Pin_Header_Straight_2x05
- removed P7: ADC(NC), Pin_Headers:Pin_Header_Straight_1x03
- added D6: BAT54-04, TO_SOT_Packages_SMD:SOT-23, B.Cu at (93.2, 139.2)
- P1: footprint Connect:bornier4 -> Connect:bornier2
- P5: value DS18b20_2 -> LED_DIMM; footprint Connect:bornier3 -> Connect:bornier2
- R11, R12: moved to B.Cu
- W1, W2, W3, W4: value TEST_1P -> HOLE
- moved JP5 62.6 mm to (108.5, 159.7)
- moved R8 58.8 mm to (118.1, 154.6), turned to 90 degrees
- moved JP4 57.2 mm to (98.9, 161.4), turned to 0 degrees
- moved R7 55.4 mm to (114.5, 154.5), turned to 270 degrees
- moved Q2 47.8 mm to (106.5, 164.5)
- moved P9 38.4 mm to (99.7, 91.3), turned to 180 degrees
- moved P5 28.7 mm to (91.6, 163.7), turned to 0 degrees
- moved P6 28.3 mm to (49.2, 159.2)
- moved D1 26.2 mm to (40.2, 114.2), turned to 270 degrees
- moved D3 23.9 mm to (93.2, 149.6), turned to 90 degrees
- moved D4 19.4 mm to (93.2, 146.1), turned to 90 degrees
- moved R10 18.3 mm to (77.9, 157.9)
- moved JP3 17.6 mm to (64.5, 157.0)
- moved RLY1 17.2 mm to (44.3, 114.2), turned to 0 degrees
- moved JP2 15.4 mm to (61.0, 147.8), turned to 270 degrees
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Connections:
- P5 pad 1: +3V3 -> DIM+
- P5 pad 2: DS18b20 -> DIM-
- R11 pad 2: Net-(F2-Pad2) -> LED1+
- R12 pad 2: LED1+ -> Net-(F2-Pad2)
- RLY1 pad 5: Net-(RLY1-Pad5) -> (no net)
- U3 pad 1: Net-(U3-Pad1) -> (no net)
- U3 pad 12: Net-(U3-Pad12) -> (no net)
- U3 pad 13: Net-(U3-Pad13) -> (no net)
- U3 pad 2: Net-(U3-Pad2) -> (no net)
- U3 pad 3: Net-(U3-Pad3) -> (no net)
- U3 pad 4: Net-(U3-Pad4) -> (no net)
- U3 pad 5: Net-(U3-Pad5) -> (no net)
- U3 pad 6: Net-(U3-Pad6) -> (no net)
- U3 pad 7: Net-(U3-Pad7) -> (no net)
- U3 pad 8: Net-(U3-Pad8) -> (no net)
- U3 pad 9: Net-(U3-Pad9) -> (no net)
- U5 pad 2: ADC_LED_COMON -> (no net)
- U5 pad 3: ADC_LED2_IN- -> ADC_LED_COMON
- U5 pad 4: Net-(P7-Pad3) -> (no net)
- U5 pad 5: Net-(P7-Pad2) -> ADC_LED2_IN-
- U5 pad 6: Net-(P7-Pad1) -> (no net)
- W1 pad 1: GND -> (no net)
- W2 pad 1: GND -> (no net)
- W3 pad 1: GND -> (no net)
- W4 pad 1: GND -> (no net)
Routing:
- net GND: track 0.00 -> 357.9 mm, vias 0 -> 8
- net +5V: track 0.00 -> 225.5 mm
- net +3V3: track 0.00 -> 177.8 mm, vias 0 -> 2
- net DIM+: track 0.00 -> 98.6 mm, vias 0 -> 2
- net Net-(F1-Pad1): track 0.00 -> 69.1 mm
- net ESP_PWM_OUT: track 0.00 -> 63.6 mm
- net Net-(D1-Pad2): track 0.00 -> 59.2 mm
- net LED1+: track 0.00 -> 57.0 mm
- net MCP_CS: track 0.00 -> 51.8 mm
- net MCP_DIN: track 0.00 -> 50.6 mm
- net MCP_DOUT: track 0.00 -> 49.3 mm
- net Net-(P2-Pad1): track 0.00 -> 49.2 mm
- net MCP_CLK: track 0.00 -> 48.8 mm
- net LED2-: track 9.81 -> 55.1 mm
- net ADC_LED2_IN-: track 0.00 -> 44.3 mm
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- added copper zone on B.Cu, net GND
Other:
- net class ADC: via_dia 0.6 -> 1.5; via_drill 0.4 -> 1
- net class Default: via_dia 0.6 -> 1.5; via_drill 0.4 -> 1
- net class HV_LED: clearance 0.5 -> 0.45
- net class LV_DC: via_dia 0.6 -> 1.5; via_drill 0.4 -> 1

Commit message: pierwszy druk
Parts:
- removed R11, R12: 0, Resistors_SMD:R_0603
- D1: footprint Discret:D3 -> Discret:D4
- U3: moved to B.Cu
- moved P8 38.9 mm to (90.9, 81.5), turned to 0 degrees
- moved U3 37.4 mm to (118.2, 82.0)
- moved R2 22.2 mm to (98.8, 90.2), turned to 90 degrees
- moved C10 18.8 mm to (106.5, 134.5), turned to 270 degrees
- moved P9 18.7 mm to (99.8, 110.0), turned to 0 degrees
- moved C3 18.0 mm to (85.0, 89.0), turned to 270 degrees
- moved C9 14.0 mm to (103.6, 136.9), turned to 90 degrees
- moved C5 10.5 mm to (74.0, 108.5), turned to 0 degrees
- moved R1 10.4 mm to (84.6, 106.4), turned to 0 degrees
- moved C2 6.52 mm to (84.5, 97.5)
- moved U2 6.47 mm to (78.0, 95.0)
- moved C8 6.07 mm to (84.5, 130.0), turned to 270 degrees
- moved JP1 5.70 mm to (73.2, 134.6), turned to 270 degrees
- moved C7 5.46 mm to (82.5, 125.0)
- moved P1 4.84 mm to (30.7, 147.3)
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Connections:
- U1 pad 1: Net-(R11-Pad1) -> Net-(F2-Pad2)
- U1 pad 2: Net-(R11-Pad1) -> Net-(F2-Pad2)
- U1 pad 3: Net-(R12-Pad1) -> LED1+
- U1 pad 4: Net-(R12-Pad1) -> LED1+
- U5 pad 1: ADC_LED1_IN+ -> LED_Current
- U5 pad 2: (no net) -> ESP_PWM_OUT
- U5 pad 3: ADC_LED_COMON -> (no net)
- U5 pad 4: (no net) -> ADC_LED2_IN-
- U5 pad 5: ADC_LED2_IN- -> (no net)
- U5 pad 6: (no net) -> ADC_LED_COMON
- U5 pad 7: ESP_PWM_OUT -> (no net)
- U5 pad 8: LED_Current -> ADC_LED1_IN+
Routing:
- net GND: track 357.9 -> 425.1 mm, vias 8 -> 0
- net DIM+: track 98.6 -> 144.1 mm
- net ESP_PWM_OUT: track 63.6 -> 100.8 mm
- net DS18b20: track 41.6 -> 71.7 mm, vias 2 -> 0
- net Net-(Q1-Pad2): track 43.1 -> 17.5 mm, vias 2 -> 0
- net MCP_CLK: track 48.8 -> 65.9 mm
- net MCP_DOUT: track 49.3 -> 65.2 mm
- net +5V: track 225.5 -> 240.2 mm
- net LED_ON: track 3.99 -> 17.3 mm
- net MCP_DIN: track 50.6 -> 63.5 mm
- net Net-(F2-Pad2): track 22.5 -> 34.7 mm
- net MCP_CS: track 51.8 -> 60.1 mm
- net LED1+: track 57.0 -> 64.0 mm
- net Net-(D1-Pad2): track 59.2 -> 63.7 mm
- net LED2-: track 55.1 -> 50.7 mm
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Other:
- net class ADC: via_dia 1.5 -> 2.2
- net class Default: via_dia 1.5 -> 2.2
- net class LV_DC: via_dia 1.5 -> 2

Commit message: board_1_0
Parts:
- added JP6: JUMPER, Pin_Headers:Pin_Header_Straight_1x02, F.Cu at (101.5, 157.1)
- moved R1 1.80 mm to (82.8, 106.5)
- moved JP5 1.61 mm to (110.1, 159.7)
- moved C5 1.11 mm to (72.9, 108.6)
- moved C6 0.84 mm to (82.2, 129.8)
- moved U1 0.79 mm to (77.1, 128.6)
- moved C7 0.79 mm to (82.8, 125.8)
- moved C8 0.79 mm to (84.8, 130.8)
- moved JP1 0.79 mm to (73.4, 135.4)
- moved W3 0.63 mm to (117.1, 165.7)
- moved W2 0.59 mm to (28.1, 165.7)
- moved W4 0.35 mm to (117.1, 77.7)
- moved W1 0.27 mm to (28.1, 77.7)
Connections:
- C3 pad 1: DIM+ -> +10V
- C4 pad 1: DIM+ -> +10V
- U2 pad 3: DIM+ -> +10V
- U4 pad 3: DIM+ -> +10V
Routing:
- net +10V: track 0.00 -> 137.7 mm, vias 0 -> 2
- net DIM+: track 144.1 -> 27.5 mm, vias 2 -> 0
- net Earth_Protective: track 37.7 -> 83.8 mm
- net GND: track 425.1 -> 393.0 mm
- net MCP_DOUT: track 65.2 -> 59.7 mm
- net Net-(D1-Pad2): track 63.7 -> 58.9 mm
- net +5V: track 240.2 -> 235.6 mm
- net MCP_DIN: track 63.5 -> 59.1 mm
- net Net-(F2-Pad2): track 34.7 -> 30.8 mm
- net Net-(JP5-Pad2): track 8.61 -> 5.26 mm
- net DS18b20: track 71.7 -> 73.4 mm
- net MCP_CLK: track 65.9 -> 64.2 mm
- net DIM-: track 12.0 -> 13.7 mm
- net Net-(Q1-Pad2): track 17.5 -> 16.0 mm
- net +3V3: track 176.9 -> 178.3 mm
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Other:
- net class ADC: clearance 0.35 -> 0.4; via_drill 1 -> 0.8
- net class Default: clearance 0.2 -> 0.4; trace_width 0.5 -> 0.7; via_drill 1 -> 0.8
- net class HV_LED: clearance 0.45 -> 0.5
- net class LV_DC: clearance 0.35 -> 0.4; via_drill 1 -> 0.8
- net class Other added: clearance 0.4, trace_width 0.7, via_dia 2.2, via_drill 0.8
- rule trace_clearance: 0.2 -> 0.4

Commit message: swieci da sie sciemniac plytka nazywa sie new costam
Parts:
- U3: moved to F.Cu
- U5: footprint Housings_SOIC:SOIC-16_7.5x10.3mm_Pitch1.27mm -> Housings_SOIC:SOIC-16_3.9x9.9mm_Pitch1.27mm
- moved U3 38.2 mm to (121.8, 120.0)
- moved U5 1.04 mm to (100.6, 144.0)
Routing:
- net GND: track 393.0 -> 193.0 mm
- net +3V3: track 178.3 -> 32.7 mm, vias 6 -> 0
- net (no net): track 0.00 -> 101.4 mm, vias 0 -> 1
- net ESP_PWM_OUT: track 100.6 -> 0.00 mm
- net +5V: track 235.6 -> 162.6 mm
- net DS18b20: track 73.4 -> 1.80 mm
- net MCP_CLK: track 64.2 -> 0.00 mm
- net MCP_DOUT: track 59.7 -> 0.00 mm
- net MCP_CS: track 59.3 -> 0.00 mm
- net MCP_DIN: track 59.1 -> 0.00 mm
- net +10V: track 137.7 -> 96.0 mm
- net LED1+: track 62.6 -> 21.8 mm
- net Net-(F2-Pad2): track 30.8 -> 71.7 mm
- net ADC_LED2_IN-: track 47.1 -> 6.86 mm
- net ADC_LED_COMON: track 39.0 -> 9.60 mm
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- removed copper zone on B.Cu, net GND
