File: kicad/plytka_0_1.sch (KiCad schematic (older format))
At the start: 31 parts

Commit message: power supply
Parts:
- removed R? (x4): R, symbol R
- removed U?: Step_up, symbol Step_up
- removed U?: IRM-05-5, CONV_IRM-05-5, symbol IRM-05-5
- added 100n: C, symbol C
- added 22u, 470u: CP, symbol CP
- added D?: Diode_Bridge, symbol Diode_Bridge
- added D?: ZENER, symbol ZENER
- added P? (x2): CONN_01X02, symbol CONN_01X02
- added R?: R, symbol R
- added T?: TRANSFO, symbol TRANSFO
- added U?: TLE_4266, SOT-223, symbol TLE_4266
- R?: value R -> 4k7
- gave numbers to parts that had none: 2
Connections:
- net labels added: +10V, ADC_LED1_IN+, ADC_LED1_IN-, ADC_LED2_IN+, ADC_LED2_IN-, LED_ON
- net labels removed: V_LAMP1, V_LAMP2, V_PWM
- wire segments 97 -> 134
- no-connect marks 0 -> 12
Other:
- note removed: "Tutaj bedzie polaczenie GND, czy to nie problem?"
- moved on the sheet: F?, P?, Q?, R?, U?

Commit message: almost ready. time for choosing footprint. still no ADC
Parts:
- removed D?: ZENER, symbol ZENER
- removed R?: R, symbol R
- added C4: 10u, symbol CP
- added C5: 100u, symbol CP
- added D3, D4: ZENER, symbol ZENER
- added P10: LV_POWER, symbol CONN_02X05
- added R3, R4, R5, R6: R, symbol R
- added U4: LD1117S50TR, TO_SOT_Packages_SMD:SOT-223, symbol LD1117S50TR
- C1: renamed from 470u; value CP -> 470u
- C2, C7: renamed from 100n; value C -> 100n
- C3: renamed from 22u; value CP -> 22u
- C6: renamed from 1n; value C -> 1n
- P1: renamed from P?; value CONN_01X02 -> LED_SUPPY
- P8: renamed from P?; value CONN_01X02 -> ESP_PINs
- P9: renamed from P?; value CONN_01X02 -> ESP_PINS2
- Q2: renamed from Q?; footprint TO-220 -> Power_Integrations:TO-220
- U2: renamed from U?; footprint SOT-223 -> TO_SOT_Packages_SMD:SOT-223
- gave numbers to parts that had none: 23
Connections:
- wire segments 134 -> 161
- no-connect marks 12 -> 14
Other:
- moved on the sheet: JP1, JP2, P11, P6, P7, P8, P9, Q2, R7, R8, U3

Commit message: ready for review
Parts:
- removed D3, D4: ZENER, symbol ZENER
- removed P11: DIMM, symbol CONN_01X02
- removed P6: LED1, symbol CONN_01X02
- removed Q1: Q_NPN_BCE, symbol Q_NPN_BCE
- removed R3, R4, R5, R6: R, symbol R
- added C8: NC, Capacitors_ThroughHole:C_Disc_D6_P5, symbol C
- added JP3, JP4: JUMPER(NC), Pin_Headers:Pin_Header_Straight_1x02, symbol JUMPER
- added P6: LEDs, Connect:bornier4, symbol CONN_01X04
- added Q1: BC548, TO_SOT_Packages_THT:TO-92_Inline_Wide, symbol BC548
- C1: footprint (none) -> Capacitors_ThroughHole:C_Radial_D8_L13_P3.8
- C2, C6, C7: footprint (none) -> Capacitors_ThroughHole:C_Disc_D6_P5
- C3: footprint (none) -> Capacitors_ThroughHole:C_Radial_D5_L6_P2.5
- C4: footprint (none) -> Capacitors_ThroughHole:C_Radial_D5_L11_P2.5
- C5: footprint (none) -> Capacitors_ThroughHole:C_Radial_D6.3_L11.2_P2.5
- D1: value D -> 1N4148; footprint (none) -> Discret:D3
- D2: footprint (none) -> w_pth_diodes:bridge_wob
- F1, F2: footprint (none) -> Fuse_Holders_and_Fuses:Fuseholder5x20_horiz_open_inline_Type-I
- JP1, JP2: value JUMPER -> JUMPER(NC); footprint (none) -> Pin_Headers:Pin_Header_Straight_1x02
- P1: footprint (none) -> Connect:bornier4; symbol CONN_01X02 -> CONN_01X04
- P10: footprint (none) -> Pin_Headers:Pin_Header_Straight_2x05
- P2, P3: footprint (none) -> Connect:bornier3; symbol CONN_01X02 -> CONN_01X03
- P4, P5: footprint (none) -> Connect:bornier3
- P7: value LED2 -> ADC(NC); footprint (none) -> Pin_Headers:Pin_Header_Straight_1x02
- P8: value ESP_PINs -> ESP_PIN1(NC); footprint (none) -> Pin_Headers:Pin_Header_Straight_1x02
- P9: value ESP_PINS2 -> ESP_PINS2(NC); footprint (none) -> Pin_Headers:Pin_Header_Straight_1x02
- Q2: value IRF540N -> IRL540N
- R1: value R -> 4k7; footprint (none) -> Discret:R5
- R2, R7, R8: footprint (none) -> Discret:R5
- RLY1: footprint (none) -> Relays_ThroughHole:Relay_SANYOU_SRD_Series_Form_C
- T1: footprint (none) -> Transformers_CHK:Trafo_CHK-EI30-2VA_Neutral
- U1: footprint SOIC127P600X175-8N -> Housings_SOIC:SOIC-8_3.9x4.9mm_Pitch1.27mm
- U3: footprint (none) -> nodemcu:NodeMCU_Amica_R2
- U5: value MCP3008 -> MCP3208; footprint (none) -> Housings_SOIC:SOIC-16_7.5x10.3mm_Pitch1.27mm; symbol MCP3008 -> MCP3008-RESCUE-plytka_0_1
Connections:
- net labels added: DIM+, DIM-, Earth_Protective, LED1+, LED1-, LED2+, LED2-
- wire segments 161 -> 178
- no-connect marks 14 -> 12
Other:
- moved on the sheet: C6, C7, D1, F1, F2, P4, P5, R1, R2, RLY1, U1

Commit message: schematic ready, board placed no routes
Parts:
- added C10, C9: 100n, Capacitors_ThroughHole:C_Disc_D3_P2.5, symbol C
- added D3, D4, D5: BAT54-04, TO_SOT_Packages_SMD:SOT-23, symbol D_Schottky_x2_Serial_AKC
- added JP5: JUMPER3, Pin_Headers:Pin_Header_Straight_1x03, symbol JUMPER3
- added R10, R5: (NC), Discret:R4, symbol R
- added R11, R12: 0, Resistors_SMD:R_0603, symbol R
- added R3, R4: 100k, Discret:R4, symbol R
- added R6: 3k, Discret:R5, symbol R
- added R9: 5k, Discret:R4, symbol R
- added W1, W2, W3, W4: TEST_1P, Connect:1pin, symbol TEST_1P
- C2, C7, C8: footprint Capacitors_ThroughHole:C_Disc_D6_P5 -> Capacitors_ThroughHole:C_Disc_D3_P2.5
- JP4: value JUMPER(NC) -> JUMPER
- P7: footprint Pin_Headers:Pin_Header_Straight_1x02 -> Pin_Headers:Pin_Header_Straight_1x03; symbol CONN_01X02 -> CONN_01X03
- R1, R2, R7, R8: footprint Discret:R5 -> Discret:R4
- T1: symbol TRANSFO -> TRANSFO-RESCUE-plytka_0_1
Connections:
- net labels added: ADC_LED_COMON
- net labels removed: ADC_LED1_IN-, ADC_LED2_IN+
- wire segments 178 -> 196
Other:
- moved on the sheet: C6, C8, JP1, JP2, JP3, P8, P9, Q2, R7, R8, U1, U3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

Commit message: almost final PCB
Parts:
- removed P10: LV_POWER, Pin_Headers:Pin_Header_Straight_2x05, symbol CONN_02X05
- removed P5: DS18b20_2, Connect:bornier3, symbol CONN_01X03
- removed P7: ADC(NC), Pin_Headers:Pin_Header_Straight_1x03, symbol CONN_01X03
- added D6: BAT54-04, TO_SOT_Packages_SMD:SOT-23, symbol D_Schottky_x2_Serial_AKC
- added P5: LED_DIMM, Connect:bornier2, symbol CONN_01X02
- P1: footprint Connect:bornier4 -> Connect:bornier2; symbol CONN_01X04 -> CONN_01X02
- W1, W2, W3, W4: value TEST_1P -> HOLE
Connections:
- wire segments 196 -> 174
- no-connect marks 12 -> 20
Other:
- moved on the sheet: F2, P6, R2

Commit message: pierwszy druk
Parts:
- removed R11, R12: 0, Resistors_SMD:R_0603, symbol R
- U4: symbol LD1117S50TR -> LD1117S50TR-RESCUE-plytka_0_1
Connections:
- wire segments 174 -> 171
Other:
- moved on the sheet: C6, C7, C8, F2
Changed lines of the file:
@@
 L VAA #PWR05
 U 1 1 5BE9D815
-P 3100 1350
-F 0 "#PWR05" H 3100 1200 50  0001 C CNN
-F 1 "VAA" H 3100 1500 50  0000 C CNN
-F 2 "" H 3100 1350 50  0000 C CNN
-F 3 "" H 3100 1350 50  0000 C CNN
-	1    3100 1350
+P 3200 1150
+F 0 "#PWR05" H 3200 1000 50  0001 C CNN
+F 1 "VAA" H 3200 1300 50  0000 C CNN
+F 2 "" H 3200 1150 50  0000 C CNN
+F 3 "" H 3200 1150 50  0000 C CNN
+	1    3200 1150
 	-1   0    0    -1
 $EndComp
@@
 L FUSE F2
 U 1 1 5BE9D875
-P 3100 1700
-F 0 "F2" H 3200 1750 50  0000 C CNN
-F 1 "FUSE" H 3000 1650 50  0000 C CNN
-F 2 "Fuse_Holders_and_Fuses:Fuseholder5x20_horiz_open_inline_Type-I" H 3100 1700 50  0001 C CNN
-F 3 "" H 3100 1700 50  0000 C CNN
-	1    3100 1700
+P 3200 1500
+F 0 "F2" H 3300 1550 50  0000 C CNN
+F 1 "FUSE" H 3100 1450 50  0000 C CNN
+F 2 "Fuse_Holders_and_Fuses:Fuseholder5x20_horiz_open_inline_Type-I" H 3200 1500 50  0001 C CNN
+F 3 "" H 3200 1500 50  0000 C CNN
+	1    3200 1500
 	0    1    1    0
 $EndComp
-Text GLabel 3550 1100 2    60   Input ~ 0
+Text GLabel 4200 2050 0    60   Input ~ 0
 V+LAMP
 $Comp
 L C C6
 U 1 1 5BE9E45E
-P 4150 2350
-F 0 "C6" H 4175 2450 50  0000 L CNN
-F 1 "1n" H 4175 2250 50  0000 L CNN
-F 2 "Capacitors_ThroughHole:C_Disc_D6_P5" H 4188 2200 50  0001 C CNN
-F 3 "" H 4150 2350 50  0000 C CNN
-	1    4150 2350
+P 4150 2400
+F 0 "C6" H 4175 2500 50  0000 L CNN
+F 1 "1n" H 4175 2300 50  0000 L CNN
+F 2 "Capacitors_ThroughHole:C_Disc_D6_P5" H 4188 2250 50  0001 C CNN
+F 3 "" H 4150 2400 50  0000 C CNN
+	1    4150 2400
 	1    0    0    -1
 $EndComp
@@
 L GND #PWR06
 U 1 1 5BE9E52E
-P 4450 2550
-F 0 "#PWR06" H 4450 2300 50  0001 C CNN
-F 1 "GND" H 4450 2400 50  0000 C CNN
-F 2 "" H 4450 2550 50  0000 C CNN
-F 3 "" H 4450 2550 50  0000 C CNN
-	1    4450 2550
+P 4450 2600
+F 0 "#PWR06" H 4450 2350 50  0001 C CNN
+F 1 "GND" H 4450 2450 50  0000 C CNN
+F 2 "" H 4450 2600 50  0000 C CNN
+F 3 "" H 4450 2600 50  0000 C CNN
+	1    4450 2600
 	1    0    0    -1
 $EndComp
@@
 L C C7
 U 1 1 5BE9E654
-P 3950 1450
-F 0 "C7" H 3975 1550 50  0000 L CNN
-F 1 "100n" H 3975 1350 50  0000 L CNN
-F 2 "Capacitors_ThroughHole:C_Disc_D3_P2.5" H 3988 1300 50  0001 C CNN
-F 3 "" H 3950 1450 50  0000 C CNN
-	1    3950 1450
+P 3950 1350
+F 0 "C7" H 3975 1450 50  0000 L CNN
+F 1 "100n" H 3975 1250 50  0000 L CNN
+F 2 "Capacitors_ThroughHole:C_Disc_D3_P2.5" H 3988 1200 50  0001 C CNN
+F 3 "" H 3950 1350 50  0000 C CNN
+	1    3950 1350
 	0    1    1    0
 $EndComp
@@
 L GND #PWR07
 U 1 1 5BE9E73A
-P 3700 1500
-F 0 "#PWR07" H 3700 1250 50  0001 C CNN
-F 1 "GND" H 3700 1350 50  0000 C CNN
-F 2 "" H 3700 1500 50  0000 C CNN
-F 3 "" H 3700 1500 50  0000 C CNN
-	1    3700 1500
+P 3700 1400
+F 0 "#PWR07" H 3700 1150 50  0001 C CNN
+F 1 "GND" H 3700 1250 50  0000 C CNN
+F 2 "" H 3700 1400 50  0000 C CNN
+F 3 "" H 3700 1400 50  0000 C CNN
+	1    3700 1400
 	1    0    0    -1
 $EndComp
@@
 L +5V #PWR08
 U 1 1 5BE9E7BB
-P 4150 1350
-F 0 "#PWR08" H 4150 1200 50  0001 C CNN
-F 1 "+5V" H 4150 1490 50  0000 C CNN
-F 2 "" H 4150 1350 50  0000 C CNN
-F 3 "" H 4150 1350 50  0000 C CNN
-	1    4150 1350
+P 4150 1250
+F 0 "#PWR08" H 4150 1100 50  0001 C CNN
+F 1 "+5V" H 4150 1390 50  0000 C CNN
+F 2 "" H 4150 1250 50  0000 C CNN
+F 3 "" H 4150 1250 50  0000 C CNN
+	1    4150 1250
 	1    0    0    -1
 $EndComp
@@
 Text GLabel 8950 2700 2    60   Input ~ 0
 ADC_LED_COMON
+Text GLabel 11950 3250 0    60   Input ~ 0
+ADC_LED1_IN+
+Text GLabel 11950 2850 0    60   Input ~ 0
+ADC_LED2_IN-
 Text GLabel 11950 2550 0    60   Input ~ 0
-ADC_LED1_IN+
-Text GLabel 11950 2950 0    60   Input ~ 0
-ADC_LED2_IN-
-Text GLabel 11950 3250 0    60   Input ~ 0
 LED_Current
-Text GLabel 11950 3150 0    60   Input ~ 0
+Text GLabel 11950 2650 0    60   Input ~ 0
 ESP_PWM_OUT
 Text GLabel 8100 5850 2    60   Input ~ 0
@@
 Text GLabel 8100 6050 2    60   Input ~ 0
 LED_ON
-$Comp
-L ACS712ELCTR-05B-T U1
-U 1 1 5BE9DD7E
-P 5400 1750
-F 0 "U1" H 5193 2347 50  0000 L BNN
-F 1 "ACS712ELCTR-05B-T" H 5263 750 50  0000 L BNN
-F 2 "Housings_SOIC:SOIC-8_3.9x4.9mm_Pitch1.27mm" H 5400 1750 50  0001 L BNN
-F 3 "SOIC-8 Allegro MicroSystems LLC" H 5400 1750 50  0001 L BNN
-F 4 "Allegro MicroSystems LLC" H 5400 1750 50  0001 L BNN "Field4"
-F 5 "Fully Integrated, Hall Effect-Based Linear Current Sensor IC with 2.1 kVRMS Voltage Isolation and a Low-Resistance Cu..." H 5400 1750 50  0001 L BNN "Field5"
-F 6 "Unavailable" H 5400 1750 50  0001 L BNN "Field6"
-F 7 "ACS712ELCTR-05B-T" H 5400 1750 50  0001 L BNN "Field7"
-F 8 "None" H 5400 1750 50  0001 L BNN "Field8"
-	1    5400 1750
-	1    0    0    -1
-$EndComp
 NoConn ~ 7150 6450
 NoConn ~ 7150 6350
@@
 $EndComp
 $Comp
-L LD1117S50TR U4
+L LD1117S50TR-RESCUE-plytka_0_1 U4
 U 1 1 5BEC8403
 P 7800 8650
@@
 L C C8
 U 1 1 5BEE8811
-P 3900 2350
-F 0 "C8" H 3925 2450 50  0000 L CNN
-F 1 "NC" H 3925 2250 50  0000 L CNN
-F 2 "Capacitors_ThroughHole:C_Disc_D3_P2.5" H 3938 2200 50  0001 C CNN
-F 3 "" H 3900 2350 50  0000 C CNN
-	1    3900 2350
+P 3900 2400
+F 0 "C8" H 3925 2500 50  0000 L CNN
+F 1 "NC" H 3925 2300 50  0000 L CNN
+F 2 "Capacitors_ThroughHole:C_Disc_D3_P2.5" H 3938 2250 50  0001 C CNN
+F 3 "" H 3900 2400 50  0000 C CNN
+	1    3900 2400
 	1    0    0    -1
 $EndComp
@@
 	1    0    0    -1
 $EndComp
-Text GLabel 11900 2750 0    60   Input ~ 0
+Text GLabel 11950 3050 0    60   Input ~ 0
 ADC_LED_COMON
 $Comp
@@
 	1    0    0    -1
 $EndComp
-$Comp
-L R R11
-U 1 1 5BF0453A
-P 4150 1700
-F 0 "R11" V 4230 1700 50  0000 C CNN
-F 1 "0" V 4150 1700 50  0000 C CNN
-F 2 "Resistors_SMD:R_0603" V 4080 1700 50  0000 C CNN
-F 3 "" H 4150 1700 50  0000 C CNN
-	1    4150 1700
-	0    1    1    0
-$EndComp
-$Comp
-L R R12
-U 1 1 5BF04887
-P 4150 1950
-F 0 "R12" V 4230 1950 50  0000 C CNN
-F 1 "0" V 4150 1950 50  0000 C CNN
-F 2 "Resistors_SMD:R_0603" V 4080 1950 50  0000 C CNN
-F 3 "" H 4150 1950 50  0000 C CNN
-	1    4150 1950
-	0    1    1    0
-$EndComp
 Wire Wire Line
 	2350 3700 2350 3600
@@
 	2600 10700 2600 10850
 Wire Wire Line
-	3100 1350 3100 1450
+	3200 1150 3200 1250
 Wire Wire Line
 	3050 10150 3050 10750
 Wire Wire Line
-	3900 2150 4700 2150
-Wire Wire Line
-	4150 2150 4150 2200
-Wire Wire Line
-	3900 2500 4700 2500
-Wire Wire Line
-	4700 2500 4700 2350
-Wire Wire Line
-	4450 2550 4450 2500
-Connection ~ 4450 2500
-Wire Wire Line
-	4100 1450 4700 1450
-Wire Wire Line
-	3700 1500 3700 1450
-Wire Wire Line
-	3700 1450 3800 1450
-Wire Wire Line
-	4150 1350 4150 1450
-Connection ~ 4150 1450
+	3900 2200 4700 2200
+Wire Wire Line
+	4150 2200 4150 2250
+Wire Wire Line
+	3900 2550 4700 2550
+Wire Wire Line
+	4450 2600 4450 2550
+Connection ~ 4450 2550
+Wire Wire Line
+	4100 1350 4700 1350
+Wire Wire Line
+	3700 1400 3700 1350
+Wire Wire Line
+	3700 1350 3800 1350
+Wire Wire Line
+	4150 1250 4150 1350
+Connection ~ 4150 1350
 Wire Wire Line
 	7000 3800 7000 4050
@@
 	3000 8450 3000 9750
 Wire Wire Line
-	4450 1650 4450 1850
-Connection ~ 4450 1700
-Wire Wire Line
-	4300 1950 4700 1950
-Wire Wire Line
-	4700 1750 4600 1750
-Wire Wire Line
-	4600 1750 4600 1950
-Connection ~ 4600 1950
-Wire Wire Line
 	8050 6350 8100 6350
 Wire Wire Line
@@
 	8450 8600 8450 8550
 Connection ~ 8350 8600
-Wire Wire Line
-	11950 3150 12050 3150
 Wire Wire Line
 	12050 3250 11950 3250
@@
 	5950 8600 5950 8450
 Connection ~ 5950 8600
-Wire Wire Line
-	3500 1100 3500 1700
 Connection ~ 3000 8450
 Wire Wire Line
@@
 Connection ~ 3050 8850
 Wire Wire Line
-	4450 1650 4700 1650
-Wire Wire Line
-	4450 1850 4700 1850
-Wire Wire Line
 	2600 10300 2600 10200
 Connection ~ 2600 10200
@@
 	3050 10750 3650 10750
 Wire Wire Line
-	3900 2150 3900 2200
-Connection ~ 4150 2150
-Connection ~ 4150 2500
+	3900 2200 3900 2250
+Connection ~ 4150 2200
+Connection ~ 4150 2550
 Wire Wire Line
 	2200 8700 2300 8700
@@
 Wire Wire Line
 	12200 2150 12250 2150
-Wire Wire Line
-	4300 1700 4450 1700
-Wire Wire Line
-	3500 1700 4000 1700
-Wire Wire Line
-	3100 1950 4000 1950
 $Comp
 L TEST_1P W1
@@
 NoConn ~ 8500 10250
 NoConn ~ 8400 10250
-NoConn ~ 12050 2850
-NoConn ~ 12050 3050
 $Comp
 L D_Schottky_x2_Serial_AKC D6
@@
 	6500 500  6500 500
 Connection ~ 6700 800
-Wire Wire Line
-	3500 1100 3550 1100
 Connection ~ 1600 3500
 Wire Wire Line
@@
 Wire Wire Line
 	11900 2750 12050 2750
-NoConn ~ 12050 2650
 NoConn ~ 13050 3300
 $Comp
@@
 	-1   0    0    -1
 $EndComp
+Wire Wire Line
+	8200 8700 8200 8600
+Connection ~ 8200 8600
+$Comp
+L ACS712ELCTR-05B-T U1
+U 1 1 5BE9DD7E
+P 5400 1750
+F 0 "U1" H 5193 2347 50  0000 L BNN
+F 1 "ACS712ELCTR-05B-T" H 5263 750 50  0000 L BNN
+F 2 "Housings_SOIC:SOIC-8_3.9x4.9mm_Pitch1.27mm" H 5400 1750 50  0001 L BNN
+F 3 "SOIC-8 Allegro MicroSystems LLC" H 5400 1750 50  0001 L BNN
+F 4 "Allegro MicroSystems LLC" H 5400 1750 50  0001 L BNN "Field4"
+F 5 "Fully Integrated, Hall Effect-Based Linear Current Sensor IC with 2.1 kVRMS Voltage Isolation and a Low-Resistance Cu..." H 5400 1750 50  0001 L BNN "Field5"
+F 6 "Unavailable" H 5400 1750 50  0001 L BNN "Field6"
+F 7 "ACS712ELCTR-05B-T" H 5400 1750 50  0001 L BNN "Field7"
+F 8 "None" H 5400 1750 50  0001 L BNN "Field8"
+	1    5400 1750
+	1    0    0    -1
+$EndComp
+Wire Wire Line
+	4700 1700 4700 1800
+Wire Wire Line
+	4700 2100 4700 2000
+Wire Wire Line
+	4200 2050 4700 2050
+Wire Wire Line
+	3200 1750 4700 1750
+Connection ~ 4700 1750
+Connection ~ 4700 2050
+Wire Wire Line
+	4700 2550 4700 2450
+Wire Wire Line
+	4700 2200 4700 2300
+Wire Wire Line
+	11950 2650 12050 2650
+Wire Wire Line
+	11950 2850 12050 2850
+Wire Wire Line
+	11950 3050 12050 3050
+NoConn ~ 12050 3150
+NoConn ~ 11950 2950
+NoConn ~ 11900 2750
 $EndSCHEMATC

Commit message: board_1_0
Parts:
- added JP6: JUMPER, Pin_Headers:Pin_Header_Straight_1x02, symbol JUMPER
Connections:
- net +10V: now also JP6.2; no longer JP5.1, P5.1 (P1)
- new net DIM+: JP5.1, JP6.1, P5.1 (P1)
Other:
- moved on the sheet: C1, C10, C2, C3, C4, C5, C6, C7, C8, C9, D1, D2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

Commit message: swieci da sie sciemniac plytka nazywa sie new costam
Parts:
- removed JP4, JP6: JUMPER, Pin_Headers:Pin_Header_Straight_1x02, symbol JUMPER
- removed JP5: JUMPER3, Pin_Headers:Pin_Header_Straight_1x03, symbol JUMPER3
- removed P2: 230V, Connect:bornier3, symbol CONN_01X03
- removed P3: MEAN_WELL, Connect:bornier3, symbol CONN_01X03
- added C11, C12, C13, C14, C15: 100n, Capacitors_SMD:C_0805, symbol C
- added P2: 230V, Connect:bornier2, symbol CONN_01X02
- added P3: MEAN_WELL, Connect:bornier2, symbol CONN_01X02
- C10, C2, C7, C9: footprint Capacitors_ThroughHole:C_Disc_D3_P2.5 -> Capacitors_SMD:C_0805
- R10: value (NC) -> 10k
- U5: footprint Housings_SOIC:SOIC-16_7.5x10.3mm_Pitch1.27mm -> Housings_SOIC:SOIC-16_3.9x9.9mm_Pitch1.27mm
Connections:
- net DIM- is gone; now on net GND: P5.2 (P2)
- net +10V: now also R10.1
- net ADC_LED1_IN+: now also U5.6 (CH5), C12.1; no longer U5.8 (CH7)
- net ADC_LED2_IN-: now also U5.2 (CH1), C14.1; no longer R10.2, U5.4 (CH3)
- net ADC_LED_COMON: now also U5.4 (CH3), C13.1; no longer U5.6 (CH5)
- net DIM+: now also Q2.2 (D), R10.2
- net ESP_PWM_OUT: now also U3.26 (D4), U5.1 (CH0), C15.1; no longer U3.28 (D2), U5.2 (CH1)
- net GND: now also C11.2, C12.2, C13.2, C14.2, C15.2; no longer R10.1, U2.2 (INH)
- net LED1+: now also U1.1 (IP+_2), U1.2 (IP+); no longer U1.3 (IP-), U1.4 (IP-_2)
- net LED_Current: now also U5.8 (CH7), C11.1; no longer U5.1 (CH0)
- net LED_ON: now also U3.28 (D2); no longer U3.26 (D4)
- net at T1.5 (AB): now also P2.2 (P2), P3.2 (P2)
- net at F1.1: now also P2.1 (P1)
- net at RLY1.3: now also P3.1 (P1)
- new net: F2.2, U1.3 (IP-), U1.4 (IP-_2)
- no-connect marks 20 -> 19
Other:
- moved on the sheet: P6
