File: kicad_v2/v2.sch (KiCad schematic (older format))
At the start: 106 parts, among them P1 ESP_RX_TX, P10 LED_conf1, P11 LED_conf2, P12 CONN_01X01, P13 CONN_01X01, P14 CONN_01X01, P15 CONN_01X01, P2 CON_MEANWELL_VDC, P3 CON_LED1, P4 CON_DIM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

Commit message: new version
Parts:
- added C32: 470u, Capacitors_ThroughHole:C_Radial_D10_L21_P5, symbol CP
- C1: value 10u -> 100u; footprint Capacitors_Tantalum_SMD:TantalC_SizeB_EIA-3528_Reflow -> Capacitors_SMD:c_elec_6.3x5.3
Connections:
- net DAC_SCL: now also U3.14 (D1); no longer U3.11 (D4)
- net DAC_SDA: now also U3.13 (D2); no longer U3.12 (D3)
- net DS18B20: now also U3.12 (D3); no longer U3.14 (D1)
- net GND: now also C32.2
- net LED1+: now also JP1.2; no longer R11.2, R13.2
- net LED_Current_meas_in: now also R11.1, R12.2; no longer JP1.1
- net LED_ON: now also U3.11 (D4); no longer U3.13 (D2)
- net at C5.1, C7.1, JP2.1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: now also C32.1
- new net: JP1.1, R11.2, R13.2
Other:
- note removed: "ten trzeba jeszcze obliczyc, zależy od spadku napiec na PNP"
- moved on the sheet: JP1, JP2
Changed lines of the file:
@@
 Text GLabel 8600 5700 0    60   Input ~ 0
 LED_Current_meas_in
-Text GLabel 8600 6800 0    60   Input ~ 0
+Text GLabel 8550 7400 0    60   Input ~ 0
 LED_Current_meas_out
 $Comp
@@
 P 950 2100
 F 0 "C1" H 975 2200 50  0000 L CNN
-F 1 "10u" H 975 2000 50  0000 L CNN
-F 2 "Capacitors_Tantalum_SMD:TantalC_SizeB_EIA-3528_Reflow" H 988 1950 50  0001 C CNN
+F 1 "100u" H 975 2000 50  0000 L CNN
+F 2 "Capacitors_SMD:c_elec_6.3x5.3" H 988 1950 50  0001 C CNN
 F 3 "" H 950 2100 50  0000 C CNN
 	1    950  2100
@@
 L +3.3V #PWR020
 U 1 1 5C6DB440
-P 3250 1900
-F 0 "#PWR020" H 3250 1750 50  0001 C CNN
-F 1 "+3.3V" H 3250 2040 50  0000 C CNN
-F 2 "" H 3250 1900 50  0000 C CNN
-F 3 "" H 3250 1900 50  0000 C CNN
-	1    3250 1900
+P 3700 1900
+F 0 "#PWR020" H 3700 1750 50  0001 C CNN
+F 1 "+3.3V" H 3700 2040 50  0000 C CNN
+F 2 "" H 3700 1900 50  0000 C CNN
+F 3 "" H 3700 1900 50  0000 C CNN
+	1    3700 1900
 	1    0    0    -1
 $EndComp
@@
 	1    0    0    -1
 $EndComp
-Text GLabel 3800 8500 2    60   Input ~ 0
+Text GLabel 3800 8700 2    60   Input ~ 0
 LED_ON
 Text GLabel 2800 8500 0    60   Input ~ 0
@@
 Text GLabel 2800 8800 0    60   Input ~ 0
 ADC_CS
+Text GLabel 3800 8500 2    60   Input ~ 0
+DAC_SDA
+Text GLabel 3800 8400 2    60   Input ~ 0
+DAC_SCL
 Text GLabel 3800 8600 2    60   Input ~ 0
-DAC_SDA
-Text GLabel 3800 8700 2    60   Input ~ 0
-DAC_SCL
-Text GLabel 3800 8400 2    60   Input ~ 0
 DS18B20
 $Comp
@@
 L JUMPER JP1
 U 1 1 5C733CE7
-P 8750 6000
-F 0 "JP1" H 8750 6150 50  0000 C CNN
-F 1 "JUMPER" H 8750 5920 50  0000 C CNN
-F 2 "Pin_Headers:Pin_Header_Straight_1x02" H 8750 6000 50  0001 C CNN
-F 3 "" H 8750 6000 50  0000 C CNN
-	1    8750 6000
+P 8750 7100
+F 0 "JP1" H 8750 7250 50  0000 C CNN
+F 1 "JUMPER" H 8750 7020 50  0000 C CNN
+F 2 "Pin_Headers:Pin_Header_Straight_1x02" H 8750 7100 50  0001 C CNN
+F 3 "" H 8750 7100 50  0000 C CNN
+	1    8750 7100
 	0    1    1    0
 $EndComp
@@
 L JUMPER JP2
 U 1 1 5C74A298
-P 2950 1950
-F 0 "JP2" H 2950 2100 50  0000 C CNN
-F 1 "JUMPER" H 2950 1870 50  0000 C CNN
-F 2 "Pin_Headers:Pin_Header_Straight_1x02" H 2950 1950 50  0001 C CNN
-F 3 "" H 2950 1950 50  0000 C CNN
-	1    2950 1950
+P 3400 1950
+F 0 "JP2" H 3400 2100 50  0000 C CNN
+F 1 "JUMPER" H 3400 1870 50  0000 C CNN
+F 2 "Pin_Headers:Pin_Header_Straight_1x02" H 3400 1950 50  0001 C CNN
+F 3 "" H 3400 1950 50  0000 C CNN
+	1    3400 1950
 	1    0    0    -1
 $EndComp
@@
 	1    0    0    -1
 $EndComp
-Text Notes 800  5650 0    60   ~ 0
-ten trzeba jeszcze obliczyc, zależy od spadku napiec na PNP
 $Comp
 L GNDA #PWR067
@@
 Connection ~ 8750 6750
 Wire Wire Line
-	8600 6800 8750 6800
-Wire Wire Line
-	8750 6800 8750 6750
+	8750 6750 8750 6800
 Wire Wire Line
 	9250 3950 9250 3850
@@
 Connection ~ 950  1950
 Wire Wire Line
-	2150 1950 2650 1950
+	2150 1950 3100 1950
 Connection ~ 2300 1950
 Wire Wire Line
-	950  2250 2600 2250
+	950  2250 2900 2250
 Connection ~ 1200 2250
 Connection ~ 1750 2250
@@
 	3250 3050 3250 3000
 Wire Wire Line
-	3250 1950 3250 1900
+	3700 1950 3700 1900
 Connection ~ 2600 1950
 Wire Wire Line
@@
 	2450 5900 2450 5800
 Wire Wire Line
-	8750 6450 8750 6300
+	8750 5700 8750 6450
 Connection ~ 2650 3050
 Wire Wire Line
@@
 NoConn ~ 5600 -900
 NoConn ~ 5600 -1150
+$Comp
+L CP C32
+U 1 1 5C7C4F89
+P 2900 2100
+F 0 "C32" H 2925 2200 50  0000 L CNN
+F 1 "470u" H 2925 2000 50  0000 L CNN
+F 2 "Capacitors_ThroughHole:C_Radial_D10_L21_P5" H 2938 1950 50  0001 C CNN
+F 3 "" H 2900 2100 50  0000 C CNN
+	1    2900 2100
+	1    0    0    -1
+$EndComp
+Connection ~ 2900 1950
+Connection ~ 2600 2250
+Wire Wire Line
+	8550 7400 8750 7400
 $EndSCHEMATC

Commit message: current version
Connections:
- no-connect marks 7 -> 9
Other:
- note added: "Alternatywnie zostawic te oporniki i dac rownloegle 0.1 bocznik. \nObliczneia tabelka mail rezystory\n"
- note added: "BC mły pinout\n"
- note added: "Low side measurement\n"
- note added: "To powinno byc na wyjsciu z zasilacza, teraz jest na wejsciu\n"
- note added: "comp out moze na A0?"
- note added: "comparator jest push pull\n"
- note added: "czy LED_ON jest bezpieczny na D4? moze lepiej D0"
- note added: "tutaj powinien byc dzielnik napiecia by mierzyc jak faktycznie sterujemy"
- note added: "usunac R19\n"
- note added: "usunac R27"
- note added: "usunac lub zabezpieczyc D0 ew kanal pomiarowy na ADC\n"
- note added: "zmienic na MCP6001\n"
- note added: "zmienic przekaznik!\n"
- note added: "zmienic wartosc opornikow te saja dzielnik tylko do 1A\n"
- note added: "zmniejszyc zdecydowanie lub usunac\n\n"
Changed lines of the file:
@@
 Wire Wire Line
 	8550 7400 8750 7400
+Text Notes 2600 5700 0    60   ~ 0
+usunac R27
+Text Notes 2900 6150 0    60   ~ 0
+BC mły pinout\n
+Text Notes 11950 5950 0    60   ~ 0
+usunac R19\n
+Text Notes 15100 5850 0    60   ~ 0
+comparator jest push pull\n
+Text Notes 3150 5100 0    60   ~ 0
+zmienic przekaznik!\n
+Text Notes 11900 5300 0    60   ~ 0
+zmniejszyc zdecydowanie lub usunac\n\n
+Text Notes 2000 7900 0    60   ~ 0
+czy LED_ON jest bezpieczny na D4? moze lepiej D0
+Text Notes 13000 9050 0    60   ~ 0
+usunac lub zabezpieczyc D0 ew kanal pomiarowy na ADC\n
+NoConn ~ 2950 8400
+NoConn ~ 2950 8200
+Text Notes 750  8250 0    60   ~ 0
+comp out moze na A0?
+Text Notes 10500 6900 0    60   ~ 0
+zmienic na MCP6001\n
+Text Notes 7550 5550 0    60   ~ 0
+To powinno byc na wyjsciu z zasilacza, teraz jest na wejsciu\n
+Text Notes 7800 6350 0    60   ~ 0
+Low side measurement\n
+Text Notes 9400 7500 0    60   ~ 0
+zmienic wartosc opornikow te saja dzielnik tylko do 1A\n
+Text Notes 13850 3550 0    60   ~ 0
+tutaj powinien byc dzielnik napiecia by mierzyc jak faktycznie sterujemy
+Text Notes 9350 7700 0    60   ~ 0
+Alternatywnie zostawic te oporniki i dac rownloegle 0.1 bocznik. \nObliczneia tabelka mail rezystory\n
 $EndSCHEMATC
